Commit message: Rewire twist_mux with velocity_smoother for joystick override during Nav2

File: my_robot/urdf/my_robot.urdf.xacro (robot description, xacro)
@@ -257,4 +257,25 @@
   </joint>
   <!-- ══════════════════════════════════════════════
+       IMU (MPU6050) — 2층 판 위, base_link(바퀴축) 기준
+         x : 바퀴축보다 25mm 앞
+         y : 중심에서 오른쪽 55mm  (오른쪽 = -y)
+         z : 바닥 130mm = base_link 기준 97.5mm
+       방향은 REP-103 정렬 확인됨 (좌회전 시 gyro z 양수) → rpy 0
+  ══════════════════════════════════════════════ -->
+  <xacro:property name="imu_x" value="0.025"/>
+  <xacro:property name="imu_y" value="-0.055"/>
+  <xacro:property name="imu_z" value="0.0975"/>
+  <link name="imu_link">
+    <visual>
+      <geometry><box size="0.02 0.016 0.003"/></geometry>
+      <material name="gray"/>
+    </visual>
+  </link>
+  <joint name="imu_joint" type="fixed">
+    <parent link="base_link"/>
+    <child  link="imu_link"/>
+    <origin xyz="${imu_x} ${imu_y} ${imu_z}" rpy="0 0 0"/>
+  </joint>
+  <!-- ══════════════════════════════════════════════
        ▼ Gazebo 전용 (robot_state_publisher는 무시)
          시뮬레이션 겸용으로 유지
@@ -301,5 +322,5 @@
         </scan>
         <range>
-          <min>0.12</min>
+          <min>0.165</min>
           <max>8.0</max>
           <resolution>0.015</resolution>
@@ -323,6 +344,6 @@
   </gazebo>
   <gazebo reference="caster_back_link">
-    <mu1>0.5</mu1><mu2>0.5</mu2>
-    <kp>100000.0</kp><kd>200.0</kd>
+    <mu1>0.3</mu1><mu2>0.3</mu2>
+    <kp>100000.0</kp><kd>150.0</kd>
     <minDepth>0.001</minDepth><maxVel>0.1</maxVel>
   </gazebo>
